Commit message: tests

File: urdf/controllers/omni_drive.urdf.xacro (robot description, xacro)
@@ -2,17 +2,17 @@
   <xacro:macro name="omni_drive_controller">
     <gazebo>
-    <plugin name="object_controller" filename="libgazebo_ros_planar_move.so">
-      <ros>
-        <remapping>odom:=odom/unfiltered</remapping>
-      </ros>
-      <command_topic>cmd_vel</command_topic>
-      <odometry_topic>odom/unfiltered</odometry_topic>
-      <odometry_frame>odom</odometry_frame>
-      <odometry_rate>20.0</odometry_rate>
-      <robot_base_frame>base_footprint</robot_base_frame>
-      <publish_odom>true</publish_odom>
-      <publish_odom_tf>false</publish_odom_tf>
-    </plugin>
-  </gazebo>
+      <plugin name="object_controller" filename="libgazebo_ros_planar_move.so">
+        <ros>
+          <remapping>odom:=odom/unfiltered</remapping>
+        </ros>
+        <command_topic>cmd_vel</command_topic>
+        <odometry_topic>odom/unfiltered</odometry_topic>
+        <odometry_frame>odom</odometry_frame>
+        <odometry_rate>20.0</odometry_rate>
+        <robot_base_frame>base_footprint</robot_base_frame>
+        <publish_odom>true</publish_odom>
+        <publish_odom_tf>false</publish_odom_tf>
+      </plugin>
+    </gazebo>
   </xacro:macro>
 </robot>

File: urdf/mecanum_properties.urdf.xacro (robot description, xacro)
@@ -13,5 +13,5 @@
   <xacro:property name="wheel_torque" value="20" />
   <xacro:property name="laser_pose">
-    <origin xyz="-0.099 0.1275 0.046" rpy="0 0 1.57"/>
+    <origin xyz="-0.099 0.1275 0.146" rpy="0 0 1.57"/>
   </xacro:property>
   <xacro:property name="depth_sensor_pose">

File: urdf/robots/mecanum.urdf.xacro (robot description, xacro)
@@ -52,11 +52,11 @@
     mass="${wheel_mass}"
   />
-  <xacro:imu/>
+  <!-- <xacro:imu/> -->
   <xacro:generic_laser>
     <xacro:insert_block name="laser_pose" />
   </xacro:generic_laser>
-  <xacro:depth_sensor>
+  <!-- <xacro:depth_sensor>
     <xacro:insert_block name="depth_sensor_pose" />
-  </xacro:depth_sensor>
+  </xacro:depth_sensor> -->
   <xacro:omni_drive_controller/>
 </robot>
