Commit message: change lidar orientation

File: urdf/mecanum_properties.urdf.xacro (robot description, xacro)
@@ -13,5 +13,5 @@
   <xacro:property name="wheel_torque" value="20" />
   <xacro:property name="laser_pose">
-    <origin xyz="-0.099 0.1275 0.146" rpy="0 0 1.57"/>
+    <origin xyz="-0.099 0.1275 0.146" rpy="0 3.14 0"/>
   </xacro:property>
   <xacro:property name="depth_sensor_pose">

Commit message: again

File: urdf/mecanum_properties.urdf.xacro (robot description, xacro)
@@ -13,5 +13,5 @@
   <xacro:property name="wheel_torque" value="20" />
   <xacro:property name="laser_pose">
-    <origin xyz="-0.099 0.1275 0.146" rpy="0 3.14 0"/>
+    <origin xyz="-0.099 0.1275 0.146" rpy="0 3.14 1.57"/>
   </xacro:property>
   <xacro:property name="depth_sensor_pose">

Commit message: adjusted lidar height

File: urdf/mecanum_properties.urdf.xacro (robot description, xacro)
@@ -13,5 +13,5 @@
   <xacro:property name="wheel_torque" value="20" />
   <xacro:property name="laser_pose">
-    <origin xyz="-0.099 0.1275 0.146" rpy="0 3.14 1.57"/>
+    <origin xyz="-0.099 0.1275 0.046" rpy="0 3.14 1.57"/>
   </xacro:property>
   <xacro:property name="depth_sensor_pose">
