Commit message: fix base frames

File: urdf/mech/base.urdf.xacro (robot description, xacro)
@@ -2,4 +2,10 @@
 <robot xmlns:xacro="http://ros.org/wiki/xacro">
   <xacro:macro name="base" params="length width height mass wheel_radius wheel_pos_z">
+    <link name="world"><link>
+    <joint name="base_joint" type="fixed">
+      <origin xyz="1.5 1.0 0" rpy="0 0 0"/>
+      <parent link="world"/>
+      <child link="base_link"/>
+    </joint>
     <link name="base_footprint"/>
     <link name="base_link">

Commit message: fix urdf

File: urdf/mech/base.urdf.xacro (robot description, xacro)
@@ -2,9 +2,9 @@
 <robot xmlns:xacro="http://ros.org/wiki/xacro">
   <xacro:macro name="base" params="length width height mass wheel_radius wheel_pos_z">
-    <link name="world"><link>
+    <link name="world"></link>
     <joint name="base_joint" type="fixed">
       <origin xyz="1.5 1.0 0" rpy="0 0 0"/>
       <parent link="world"/>
-      <child link="base_link"/>
+      <child link="base_footprint"/>
     </joint>
     <link name="base_footprint"/>

Commit message: added odom link

File: urdf/mech/base.urdf.xacro (robot description, xacro)
@@ -2,8 +2,8 @@
 <robot xmlns:xacro="http://ros.org/wiki/xacro">
   <xacro:macro name="base" params="length width height mass wheel_radius wheel_pos_z">
-    <link name="world"></link>
+    <link name="odom"></link>
     <joint name="base_joint" type="fixed">
       <origin xyz="1.5 1.0 0" rpy="0 0 0"/>
-      <parent link="world"/>
+      <parent link="odom"/>
       <child link="base_footprint"/>
     </joint>

Commit message: no more odom

File: urdf/mech/base.urdf.xacro (robot description, xacro)
@@ -2,10 +2,10 @@
 <robot xmlns:xacro="http://ros.org/wiki/xacro">
   <xacro:macro name="base" params="length width height mass wheel_radius wheel_pos_z">
-    <link name="odom"></link>
+    <!-- <link name="odom"></link>
     <joint name="base_joint" type="fixed">
       <origin xyz="1.5 1.0 0" rpy="0 0 0"/>
       <parent link="odom"/>
       <child link="base_footprint"/>
-    </joint>
+    </joint> -->
     <link name="base_footprint"/>
     <link name="base_link">
